File: atlas.kicad_pcb (KiCad board)
At the start: 2 copper layers, 25 parts, among them J1 AudioJack3, J2 Micro_SD_Card, SW1 SW_Push, SW2 SW_SPST, SW3 SW_Push, SW4 SW_Push, SW5 SW_Push, SW6 SW_Push, U1 ATmega328-P, U2 DAC8571IDGK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

Commit message: Add files via upload
Parts:
- removed SW2: SW_SPST, Button_Switch_THT:SW_PUSH_6mm
- removed Y1: Crystal, Crystal:Crystal_C26-LF_D2.1mm_L6.5mm_Horizontal
- added C10: C, Capacitor_SMD:C_1808_4520Metric_Pad1.72x2.30mm_HandSolder, B.Cu at (140.8, 73.7)
- added C11: C, Capacitor_SMD:C_1808_4520Metric_Pad1.72x2.30mm_HandSolder, B.Cu at (140.8, 77.5)
- added C12: C, Capacitor_SMD:C_1808_4520Metric_Pad1.72x2.30mm_HandSolder, B.Cu at (119.2, 80.8)
- added C13: C, Capacitor_SMD:C_1808_4520Metric_Pad1.72x2.30mm_HandSolder, B.Cu at (123.0, 80.8)
- added C7: C, Capacitor_SMD:C_1808_4520Metric_Pad1.72x2.30mm_HandSolder, B.Cu at (136.3, 82.0)
- added C8: C, Capacitor_SMD:C_1808_4520Metric_Pad1.72x2.30mm_HandSolder, B.Cu at (140.8, 66.0)
- added C9: C, Capacitor_SMD:C_1808_4520Metric_Pad1.72x2.30mm_HandSolder, B.Cu at (140.8, 69.8)
- added R6: R, Resistor_SMD:R_0201_0603Metric, B.Cu at (145.7, 77.0)
- added R7: R, Resistor_SMD:R_0201_0603Metric, B.Cu at (145.7, 78.8)
- added R8: R, Resistor_SMD:R_0201_0603Metric, B.Cu at (145.7, 80.5)
- added R9: R, Resistor_SMD:R_0201_0603Metric, B.Cu at (145.7, 82.2)
- added U6: LM386, Package_DIP:DIP-8_W7.62mm, B.Cu at (157.3, 101.7)
- J2: moved to B.Cu
- U1: value ATmega328-P -> PCM5122PW; footprint Package_DFN_QFN:HVQFN-32-1EP_5x5mm_P0.5mm_EP3.1x3.1mm -> Package_SO:TSSOP-28_4.4x9.7mm_P0.65mm
- U2: value DAC8571IDGK -> ESP32-WROOM-32; footprint Package_SO:MSOP-8_3x3mm_P0.65mm -> RF_Module:ESP32-WROOM-32
- U4: value NE5532 -> LM386; footprint Package_CSP:LFCSP-8_2x2mm_P0.5mm -> Package_DIP:DIP-8_W7.62mm
- moved SW1 54.7 mm to (103.8, 117.8)
- moved SW6 48.3 mm to (146.0, 118.0)
- moved J1 47.7 mm to (108.5, 73.5)
- moved SW5 41.7 mm to (135.5, 118.0)
- moved SW3 40.6 mm to (114.5, 118.0)
- moved SW4 38.9 mm to (125.0, 118.0)
- moved U2 30.3 mm to (137.7, 95.1)
- moved J2 26.7 mm to (118.3, 92.3), turned to 90 degrees
- moved C1 21.2 mm to (132.9, 66.2), turned to 180 degrees
- moved U1 19.4 mm to (148.6, 69.9), turned to 0 degrees
- moved C5 18.9 mm to (115.3, 80.8)
- moved C3 13.5 mm to (132.9, 70.0), turned to 180 degrees
- moved C2 11.2 mm to (111.5, 80.8)
- moved U4 10.2 mm to (126.3, 66.7), turned to 180 degrees
- moved RV1 8.51 mm to (119.0, 102.5), turned to 180 degrees
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Connections:
- C1 pad 1: GND -> Net-(U1-AVDD)
- C1 pad 2: Net-(C1-Pad2) -> GND
- C2 pad 1: Net-(U2-V_{SENSE}) -> Net-(U1-OUTL)
- C2 pad 2: Net-(C2-Pad2) -> GND
- C3 pad 1: Net-(U1-XTAL2/PB7) -> Net-(U1-AVDD)
- C4 pad 1: Net-(SW2-B) -> Net-(U1-AVDD)
- C4 pad 2: Net-(U1-VCC) -> GND
- C5 pad 1: Net-(SW2-B) -> Net-(U1-OUTL)
- C5 pad 2: Net-(U1-AREF) -> GND
- C6 pad 1: Net-(SW2-B) -> Net-(U6-BYPASS)
- C6 pad 2: Net-(U1-AVCC) -> GND
- J1 pad T: Net-(J1-PadR) -> Net-(J1-PadT)
- J2 pad 2: PD7 -> unconnected-(J2-DAT3/CD-Pad2)
- J2 pad 3: PD6 -> unconnected-(J2-CMD-Pad3)
- J2 pad 5: PD5 -> unconnected-(J2-CLK-Pad5)
- J2 pad 7: PD4 -> unconnected-(J2-DAT0-Pad7)
- R1 pad 1: PB1 -> unconnected-(R1-Pad1)
- R2 pad 1: PB0 -> unconnected-(R2-Pad1)
- R3 pad 1: PB2 -> unconnected-(R3-Pad1)
- R4 pad 1: PB3 -> unconnected-(R4-Pad1)
- R5 pad 1: PB4 -> unconnected-(R5-Pad1)
- RV1 pad 1: Net-(C2-Pad2) -> unconnected-(RV1-Pad1)
- RV1 pad 2: Net-(J1-PadR) -> unconnected-(RV1-Pad2)
- U1 pad 1: unconnected-(U1-~{RESET}/PC6-Pad1) -> Net-(U1-AVDD)
- U1 pad 10: Net-(U1-XTAL2/PB7) -> unconnected-(U1-VCOM/DEMP-Pad10)
- U1 pad 11: PD5 -> unconnected-(U1-SDA/MOSI/ATT2-Pad11)
- U1 pad 12: PD6 -> unconnected-(U1-SCL/MC/ATT1-Pad12)
- U1 pad 13: PD7 -> unconnected-(U1-GPIO5/ATT0-Pad13)
- U1 pad 14: PB0 -> unconnected-(U1-GPIO4/MAST-Pad14)
- U1 pad 15: PB1 -> unconnected-(U1-GPIO3/AGNS-Pad15)
- U1 pad 16: PB2 -> unconnected-(U1-ADR2/GPIO2/DOUT-Pad16)
- U1 pad 17: PB3 -> unconnected-(U1-MODE1-Pad17)
- U1 pad 18: PB4 -> unconnected-(U1-MODE2/MS-Pad18)
- U1 pad 20: Net-(U1-AVCC) -> SCK
- U1 pad 21: Net-(U1-AREF) -> BCK
- U1 pad 22: Net-(BT1--) -> DIN
- U1 pad 23: unconnected-(U1-PC0-Pad23) -> LRCK
- U1 pad 27: unconnected-(U1-PC4-Pad27) -> GND
- U1 pad 28: unconnected-(U1-PC5-Pad28) -> Net-(U1-AVDD)
- U1 pad 4: PD2 -> unconnected-(U1-CAPM-Pad4)
- U1 pad 5: PD3 -> unconnected-(U1-VNEG-Pad5)
- U1 pad 6: PD4 -> Net-(U1-OUTL)
- U1 pad 7: Net-(U1-VCC) -> Net-(U1-OUTR)
- U1 pad 8: Net-(BT1--) -> Net-(U1-AVDD)
- U1 pad 9: Net-(U1-XTAL1/PB6) -> GND
- U2 pad 1: +5V -> Net-(BT2--)
- U2 pad 2: +5V -> Net-(BT2-+)
- U2 pad 3: Net-(U2-V_{SENSE}) -> unconnected-(U2-EN-Pad3)
- U2 pad 4: Net-(U2-V_{OUT}) -> unconnected-(U2-SENSOR_VP-Pad4)
- U2 pad 5: GND -> unconnected-(U2-SENSOR_VN-Pad5)
- U2 pad 6: PD2 -> unconnected-(U2-IO34-Pad6)
- U2 pad 7: PD3 -> unconnected-(U2-IO35-Pad7)
- U2 pad 8: GND -> unconnected-(U2-IO32-Pad8)
- U3 pad 8: PD5 -> unconnected-(U3-SCLK-Pad8)
- U4 pad 1: Net-(U2-V_{SENSE}) -> unconnected-(U4-GAIN-Pad1)
- U4 pad 2: Net-(U2-V_{SENSE}) -> Net-(U1-OUTR)
- U4 pad 3: Net-(U2-V_{OUT}) -> Net-(U1-OUTR)
- U4 pad 4: (no net) -> GND
- U4 pad 5: (no net) -> Net-(C11-Pad1)
- U4 pad 6: (no net) -> +5V
- U4 pad 7: (no net) -> Net-(U4-BYPASS)
- U4 pad 8: (no net) -> unconnected-(U4-GAIN-Pad8)
Routing:
- net GND: track 200.8 -> 0.00 mm, vias 3 -> 0
- net +5V: track 164.9 -> 0.00 mm, vias 2 -> 0
- net Net-(J1-PadR): track 72.7 -> 0.00 mm, vias 1 -> 0
- net PD6: track 68.3 -> 0.00 mm, vias 3 -> 0
- net PD5: track 52.4 -> 0.00 mm, vias 4 -> 0
- net Net-(SW2-B): track 51.5 -> 0.00 mm, vias 2 -> 0
- net PD4: track 37.9 -> 0.00 mm, vias 1 -> 0
- net PD7: track 36.3 -> 0.00 mm, vias 3 -> 0
- net Net-(U1-AVCC): track 27.5 -> 0.00 mm, vias 2 -> 0
- net Net-(U1-AREF): track 26.6 -> 0.00 mm, vias 2 -> 0
- net Net-(C1-Pad2): track 23.2 -> 0.00 mm, vias 1 -> 0
- net Net-(U1-VCC): track 19.2 -> 0.00 mm
- net PD3: track 18.2 -> 0.00 mm, vias 2 -> 0
- net Net-(C2-Pad2): track 17.1 -> 0.00 mm
- net Net-(U2-V_{SENSE}): track 14.7 -> 0.00 mm
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